File: hardware/kicad files/numlocked_shift/numlocked_shift.kicad_pcb (KiCad board)
At the start: 4 copper layers, 216.5 x 140 mm, 139 parts, among them J1 Conn_01x02, J2 Conn_01x02, J3 Conn_01x04, J4 Conn_01x04, J5 Conn_01x04, J6 Conn_01x04, J7 Conn_01x04, J8 SM04B-SRSS-TB, U1 RP2040, U10 DS3231MZ, U11 74LVC1G17, U12 74LVC1G17, U13 SN74HC165DR, U2 W25Q128JVSIQ, U3 LM3940IMP-3.3/NOPB, U4 SN74HC165DR, U5 SN74HC165DR, U6 SN74HC165DR, U7 SN74HC165DR, X1 ABM8-272-T3

Commit message: Hardware V3 (changing)
Parts:
- removed BT1: Battery_Cell, numlocked_components:Q&J CR1220-2
- removed C32, C33: 0.1 uF, Capacitor_SMD:C_0603_1608Metric
- removed RN9: 10K, Resistor_SMD:R_Array_Convex_4x1206
- removed U10: DS3231MZ, Package_SO:SOIC-8_3.9x4.9mm_P1.27mm
- added S39: ~, numlocked_components:SW_Cherry_Kalih_1.00u, F.Cu at (220.5, 148.7)
- added S40: ~, numlocked_components:SW_Cherry_Kalih_1.00u, F.Cu at (151.5, 148.7)
- R11: footprint Resistor_SMD:R_0603_1608Metric -> Resistor_SMD:R_0603_1608Metric_Pad0.98x0.95mm_HandSolder
- R8: value 10k -> 1K
- moved R8 151.3 mm to (51.2, 63.5), turned to 0 degrees
- moved R4 149.4 mm to (51.2, 60.3), turned to 180 degrees
- moved C7 147.5 mm to (51.2, 61.9), turned to 180 degrees
- moved C14 146.4 mm to (48.1, 66.3), turned to 90 degrees
- moved C3 144.6 mm to (53.9, 60.9), turned to 90 degrees
- moved X1 142.8 mm to (51.0, 66.3), turned to 180 degrees
- moved C38 142.7 mm to (58.0, 57.5), turned to 180 degrees
- moved C13 138.0 mm to (53.9, 66.3), turned to 90 degrees
- moved C8 137.8 mm to (62.6, 56.1), turned to 90 degrees
- moved C9 135.6 mm to (64.2, 56.1), turned to 90 degrees
- moved U1 133.0 mm to (59.8, 62.7), turned to 90 degrees
- moved C5 132.0 mm to (66.6, 56.4), turned to 0 degrees
- moved C11 129.6 mm to (66.6, 57.9), turned to 0 degrees
- moved C6 128.7 mm to (58.8, 68.5), turned to -90 degrees
- moved C12 127.2 mm to (66.6, 59.6), turned to 0 degrees
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Connections:
- C14 pad 2: /XOUT -> Net-(C14-Pad2)
- J8 pad 1: GND -> VBUS
- J8 pad 2: /USB_RP2040+ -> /USB_RP2040-
- J8 pad 3: /USB_RP2040- -> /USB_RP2040+
- J8 pad 4: VBUS -> GND
- R8 pad 1: Net-(U1-GPIO19) -> Net-(C14-Pad2)
- R8 pad 2: +3V3 -> /XOUT
- S11 pad 1: Net-(RN3-R2.1) -> Net-(RN3-R4.1)
- S12 pad 1: Net-(RN3-R1.1) -> Net-(RN4-R4.1)
- S13 pad 1: Net-(RN4-R4.1) -> Net-(RN3-R2.1)
- S33 pad 1: Net-(U1-GPIO19) -> Net-(RN11-R2.1)
- S9 pad 1: Net-(RN3-R4.1) -> Net-(RN3-R1.1)
- U1 pad 13: unconnected-(U1-GPIO10-Pad13) -> /SH
- U1 pad 14: /Encoder B -> /CLK
- U1 pad 15: unconnected-(U1-GPIO12-Pad15) -> /rightCheckWire
- U1 pad 16: unconnected-(U1-GPIO13-Pad16) -> /numpadCheckWire
- U1 pad 2: /SSD1306 SDA -> /~{USB BOOT}
- U1 pad 27: /SH -> unconnected-(U1-GPIO16-Pad27)
- U1 pad 28: /SerialOut -> unconnected-(U1-GPIO17-Pad28)
- U1 pad 29: /CLK -> /ENC_MAIN_SW
- U1 pad 3: /SSD1306 SCL -> /SerialOut
- U1 pad 30: Net-(U1-GPIO19) -> /ENC_MAIN_B
- U1 pad 31: /~{RTC_RST} -> /ENC_MAIN_A
- U1 pad 32: /~{RTC_INT} -> unconnected-(U1-GPIO21-Pad32)
- U1 pad 34: /RTC_SDA -> /SSD1306 SDA
- U1 pad 35: /RTC_SCL -> /SSD1306 SCL
- U1 pad 36: /RTC_32KHZ -> unconnected-(U1-GPIO24-Pad36)
- U1 pad 39: /ENC_MAIN_A -> unconnected-(U1-GPIO27_ADC1-Pad39)
- U1 pad 4: /~{USB BOOT} -> /numlockLED/scrlockLED
- U1 pad 40: /ENC_MAIN_B -> unconnected-(U1-GPIO28_ADC2-Pad40)
- U1 pad 41: /ENC_MAIN_SW -> unconnected-(U1-GPIO29_ADC3-Pad41)
- U1 pad 5: /rightCheckWire -> /capsLED
- U1 pad 6: /numpadCheckWire -> /Encoder A
- U1 pad 7: /numlockLED/scrlockLED -> /Encoder B
- U1 pad 8: /capsLED -> unconnected-(U1-GPIO6-Pad8)
- U1 pad 9: /Encoder A -> unconnected-(U1-GPIO7-Pad9)
- U13 pad 10: /SerialInFromMux -> Net-(U13-SER)
- U13 pad 9: Net-(U13-QH) -> /SerialOut
- U4 pad 10: Net-(U13-QH) -> Net-(U4-SER)
- U4 pad 9: Net-(U4-QH) -> Net-(U13-SER)
- U5 pad 10: Net-(U4-QH) -> Net-(U5-SER)
- U5 pad 9: Net-(U5-QH) -> Net-(U4-SER)
- U6 pad 10: Net-(U5-QH) -> Net-(U6-SER)
- U6 pad 9: Net-(U6-QH) -> Net-(U5-SER)
- U7 pad 10: Net-(U6-QH) -> /SerialInFromMux
- U7 pad 9: /SerialOut -> Net-(U6-SER)
- X1 pad 3: /XOUT -> Net-(C14-Pad2)
Routing:
- net Net-(RN11-R3.1): track 3.59 -> 247.4 mm, vias 0 -> 2
- net /ENC_MAIN_SW: track 258.6 -> 21.2 mm, vias 2 -> 0
- net +3V3: track 627.6 -> 398.8 mm, vias 35 -> 28
- net /ENC_MAIN_A: track 238.8 -> 24.2 mm, vias 2 -> 0
- net Net-(RN11-R2.1): track 3.59 -> 211.2 mm, vias 0 -> 2
- net /ENC_MAIN_B: track 216.0 -> 27.8 mm, vias 2 -> 0
- net /SH: track 368.4 -> 190.4 mm, vias 7 -> 2
- net /numlockLED/scrlockLED: track 48.5 -> 220.5 mm, vias 0 -> 5
- net Net-(RN11-R1.1): track 3.53 -> 158.8 mm, vias 0 -> 2
- net /USB_RP2040-: track 163.9 -> 20.5 mm
- net /USB_RP2040+: track 163.2 -> 21.3 mm
- net /SerialInFromMux: track 14.6 -> 147.7 mm, vias 0 -> 2
- net Net-(RN3-R2.1): track 124.9 -> 53.9 mm
- net /numpadCheckWire: track 383.3 -> 313.3 mm, vias 1 -> 5
- net /SerialOut: track 116.4 -> 47.5 mm
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Other:
- outline, holes or cut-outs redrawn
- board text added: "Designed by YuhKuro"
- board text added: "Designed by YuhKuro Revision C"
- board text added: "Numlocked Modular Keyboard"
- board text removed: "Designed by YuhKuro Revision B"
- board text removed: "Numlocked: Shift Modular Keyboard"
