File: hardware/kicad files/numlocked_shift/numlocked_shift.kicad_sch (KiCad schematic)
At the start: 127 parts, among them J1 Conn_01x02, J2 Conn_01x02, J3 Conn_01x04, J4 Conn_01x04, J5 Conn_01x04, J6 Conn_01x04, J7 Conn_01x04, J8 AYF530435, U1 RP2040, U10 DS3231MZ, U11 74LVC1G17, U12 74LVC1G17, U13 SN74HC165DR, U2 W25Q128JVSIQ, U3 LM3940IMP-3.3/NOPB, U4 SN74HC165DR, U5 SN74HC165DR, U6 SN74HC165DR, U7 SN74HC165DR, X1 ABM8-272-T3

Commit message: Refactored file structure for hardware.
Parts:
- removed J8: AYF530435, Numlocked:AYF530435, symbol 5051100492 (Molex FFC):5051100492
- added C20, C21: 0.01 uF, Capacitor_SMD:C_0603_1608Metric, symbol Device:C
- added J8: SM04B-SRSS-TB, CONN_SM04B-SRSS-TB_JST, symbol SM04B-SRSS-TB:SM04B-SRSS-TB
- added MT1: PEC11R-4215F-S0024, PEC11R_4215F_S0024:XDCR_PEC11R-4215F-S0024, symbol PEC11R-4215F-S0024:PEC11R-4215F-S0024
- added R1, R12, R13, R14, R7: 10k, Resistor_SMD:R_0603_1608Metric, symbol Device:R
Connections:
- net +3V3: now also R14.2
- net GND: now also C20.2, C21.2, J8.1, MT1.2, MT1.COM, MT1.S1 (SHIELD), MT1.S2 (SHIELD__1)
- net USB_RP2040+: now also J8.2
- net USB_RP2040-: now also J8.3
- net VBUS: now also J8.4, R1.2, R7.2
- net ENC_MAIN_A: now reaches U1.39 (GPIO27_ADC1)
- net ENC_MAIN_A: now also C20.1, R12.1
- net ENC_MAIN_B: now reaches U1.40 (GPIO28_ADC2)
- net ENC_MAIN_B: now also C21.1, R13.1
- net ENC_MAIN_SW: now reaches U1.41 (GPIO29_ADC3)
- net ENC_MAIN_SW: now also MT1.1, R14.1
- new net: MT1.A, R1.1, R12.2
- new net: MT1.B, R13.2, R7.1
- no-connect marks 19 -> 16
Other:
- note added: "CapsLED"
- note added: "Pull Ups located on OLED PCB."
- note added: "To USB Hub Board (FFC)"
- note removed: "To USB-C Hub Board (FFC)"
- moved on the sheet: Brd1, C1, C10, C11, C12, C13, C14, C16, C17, C18, C19, C2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

Commit message: Hardware V3 (changing)
Parts:
- removed BT1: Battery_Cell, numlocked_components:Q&J CR1220-2, symbol Device:Battery_Cell
- removed C32, C33: 0.1 uF, Capacitor_SMD:C_0603_1608Metric, symbol Device:C
- removed RN9: 10K, Resistor_SMD:R_Array_Convex_4x1206, symbol Device:R_Pack04
- removed U10: DS3231MZ, Package_SO:SOIC-8_3.9x4.9mm_P1.27mm, symbol Timer_RTC:DS3231MZ
- added S39, S40: ~, numlocked_components:SW_Cherry_Kalih_1.00u, symbol Numlocked_library:SW_Cherry_KalihSocket
- J8: footprint CONN_SM04B-SRSS-TB_JST -> SM04B:CONN_SM04B-SRSS-TB_JST
- R11: footprint Resistor_SMD:R_0603_1608Metric -> Resistor_SMD:R_0603_1608Metric_Pad0.98x0.95mm_HandSolder
- R8: value 10k -> 1K
Connections:
- net RTC_SCL is gone; now on net SSD1306 SCL: U1.35 (GPIO23)
- net RTC_SDA is gone; now on net SSD1306 SDA: U1.34 (GPIO22)
- net ~{RTC_RST} is gone; now on net ENC_MAIN_A: U1.31 (GPIO20)
- net +3V3: no longer R8.2
- net CLK: now also U1.14 (GPIO11); no longer U1.29 (GPIO18)
- net ENC_MAIN_A: no longer U1.39 (GPIO27_ADC1)
- net ENC_MAIN_B: now also U1.30 (GPIO19); no longer U1.40 (GPIO28_ADC2)
- net ENC_MAIN_SW: now also U1.29 (GPIO18); no longer U1.41 (GPIO29_ADC3)
- net Encoder A: now also U1.6 (GPIO4); no longer U1.9 (GPIO7)
- net Encoder B: now also U1.7 (GPIO5); no longer U1.14 (GPIO11)
- net GND: now also J8.4, S39.2, S40.2; no longer J8.1
- net SH: now also U1.13 (GPIO10); no longer U1.27 (GPIO16)
- net SSD1306 SCL: no longer U1.3 (GPIO1)
- net SSD1306 SDA: no longer U1.2 (GPIO0)
- net SerialInFromMux: now also U7.10 (SER); no longer U13.10 (SER)
- net SerialOut: now also U1.3 (GPIO1), U13.9 (QH); no longer U1.28 (GPIO17), U7.9 (QH)
- net USB_RP2040+: now also J8.3; no longer J8.2
- net USB_RP2040-: now also J8.2; no longer J8.3
- net VBUS: now also J8.1; no longer J8.4
- net XOUT: now also R8.2; no longer C14.2, X1.3
- net capsLED: now also U1.5 (GPIO3); no longer U1.8 (GPIO6)
- net numlockLED/scrlockLED: now also U1.4 (GPIO2); no longer U1.7 (GPIO5)
- net numpadCheckWire: now also U1.16 (GPIO13); no longer U1.6 (GPIO4)
- net rightCheckWire: now also U1.15 (GPIO12); no longer U1.5 (GPIO3)
- net ~{USB BOOT}: now also U1.2 (GPIO0); no longer U1.4 (GPIO2)
- net at RN4.4 (R4.1), U5.3 (E): now also S12.1; no longer S13.1
- net at RN11.1 (R1.1), U13.6 (H): now also S40.1
- net at RN11.2 (R2.1), U13.5 (G): now also S33.1
- net at RN11.3 (R3.1), U13.4 (F): now also S39.1
- net at U6.10 (SER): now also U7.9 (QH); no longer U5.9 (QH)
- net at U6.9 (QH): now also U5.10 (SER); no longer U7.10 (SER)
- net at RN3.2 (R2.1), U5.13 (C): now also S13.1; no longer S11.1
- net at RN3.1 (R1.1), U5.14 (D): now also S9.1; no longer S12.1
- net at RN3.4 (R4.1), U5.11 (A): now also S11.1; no longer S9.1
- net at U4.9 (QH): now also U13.10 (SER); no longer U5.10 (SER)
- net at U4.10 (SER): now also U5.9 (QH); no longer U13.9 (QH)
- net RTC_32KHZ: no longer names the net of U1.36 (GPIO24)
- net ~{RTC_INT}: no longer names the net of U1.32 (GPIO21)
- new net: C14.2, R8.1, X1.3
- no-connect marks 16 -> 22
Other:
- note added: "Capslock LED"
- note added: "Encoder (leftside)"
- note removed: "Battery (CR1220)"
- note removed: "CapsLED"
- note removed: "Keyboard Switch (not enough SRs.)"
- note removed: "Pull-up Res"
- note removed: "RTC and Battery"
- note removed: "Using I2C0 SDA on GPIO0, I2C0 SCL on GPIO1"
- moved on the sheet: C20, C21, D2, MT1, R1, R11, R12, R13, R14, R7
