File: hardware/KiCad Files/numlocked_left_plate/numlocked_left_plate.kicad_pcb (KiCad board)
At the start: 2 copper layers, 216.6 x 136.8 mm, 11 parts

Commit message: Another quick hardware push. Sorry Github servers.
Other:
- outline, holes or cut-outs redrawn
