File: hardware/KiCad Files/numlocked_numpad/numlocked_numpad.kicad_pcb (KiCad board)
At the start: 4 copper layers, 81 x 139 mm, 87 parts, among them J1 Conn_01x04, J2 Conn_01x04, J3 Conn_01x04, J4 Conn_01x04, J5 Conn_01x02, J6 Conn_01x02, J7 SM04B-SRSS-TB, U1 LM3940IMP-3.3/NOPB, U2 SN74HC165DR, U3 SN74HC165DR, U4 SN74HC165DR, U6 RP2040, U7 W25Q128JVSIQ, X1 ABM8G-12.000MHZ-18-D2Y-T

Commit message: Another quick hardware push. Sorry Github servers.
Parts:
- added C1: 10 uF, Capacitor_SMD:C_0603_1608Metric, B.Cu at (95.3, 57.3)
- moved D1 29.0 mm to (122.5, 56.5), turned to 180 degrees
- moved R5 25.2 mm to (119.4, 56.5), turned to 0 degrees
- moved J6 16.6 mm to (127.5, 53.0)
- moved H1 2.00 mm to (115.0, 50.3)
- moved R3 1.66 mm to (144.7, 67.5), turned to -90 degrees
Connections:
- C11 pad 2: /XOUT -> Net-(C11-Pad2)
- R3 pad 2: /XIN -> Net-(C11-Pad2)
- X1 pad 3: /XOUT -> Net-(C11-Pad2)
Routing:
- net /~{reset}: track 7.52 -> 24.0 mm, vias 1 -> 3
- net Net-(C11-Pad2): track 0.00 -> 5.12 mm
- net /XOUT: track 8.62 -> 3.52 mm
- net +3V3: track 344.2 -> 347.9 mm
- net /SSD1112 DC: track 47.2 -> 46.6 mm
