File: hardware/KiCad Files/numlocked_numpad/numlocked_numpad.kicad_sch (KiCad schematic)
At the start: 86 parts, among them J1 Conn_01x04, J2 Conn_01x04, J3 Conn_01x04, J4 Conn_01x04, J5 Conn_01x02, J6 Conn_01x02, J7 SM04B-SRSS-TB, U1 LM3940IMP-3.3/NOPB, U2 SN74HC165DR, U3 SN74HC165DR, U4 SN74HC165DR, U6 RP2040, U7 W25Q128JVSIQ, X1 ABM8G-12.000MHZ-18-D2Y-T

Commit message: Another quick hardware push. Sorry Github servers.
Parts:
- added C1: 10 uF, Capacitor_SMD:C_0603_1608Metric, symbol Device:C
Connections:
- net +3V3: now also C1.1
- net GND: now also C1.2
- net XIN: no longer R3.2
- net XOUT: no longer C11.2, X1.3
- new net: C11.2, R3.2, X1.3
